File: HW2/PIC32board/PIC32board.sch (EAGLE design)
At the start: 25 parts

Commit message: started brd file
Parts:
- removed R3, R4: 10k, me433:10KOHM-HORIZ-1/4W-1%
- removed U$3: 0.1µF-SMD, me433:0.1µF-SMD
- added U$10: 10µF-POL, me433:10µF-POL
- added U$18: 10KOHM-SMD, me433:10KOHM-SMD
- U$12: value 10µF-POL -> 10KOHM-SMD; device me433:10µF-POL -> me433:10KOHM-SMD
Connections:
- net 5V: now also J3.2
- net B13: now also J3.6; no longer J3.3
- net B14: now also J3.7; no longer J3.2
- net B15: now also J3.8; no longer J3.1
- net B4: now also U$18.2; no longer R4.2
- net B7: now also J3.3; no longer J3.6
- net B8: now also J3.4; no longer J3.5
- net B9: now also J3.5; no longer J3.4
- net GND: now also J3.1, U$10.-; no longer J3.8, U$12.-, U$3.2
- net MCLR: now also U$12.2; no longer R3.2
- net VBUS: no longer J3.7
- net VDD: now also U$10.+, U$12.1, U$18.1; no longer R3.1, R4.1, U$12.+, U$3.1

Commit message: finished adding traces
Parts:
- renumbered U$15 to U$3
Connections:
- net A4: now also D1.C; no longer D1.A
- net N$2: now also D1.A; no longer D1.C
Other:
- moved on the sheet: D1
Changed lines of the file:
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@@
 <part name="U$13" library="me433" deviceset="BTN" device=""/>
 <part name="U$14" library="me433" deviceset="BTN" device=""/>
-<part name="D1" library="me433" deviceset="LED-GREEN" device="0603" value="GREEN"/>
 <part name="D2" library="me433" deviceset="LED-RED" device="0603" value="RED"/>
-<part name="U$15" library="me433" deviceset="MCP1702" device=""/>
 <part name="U$17" library="me433" deviceset="USB-B" device=""/>
 <part name="J1" library="me433" deviceset="CONN_06" device="SILK_FEMALE_PTH"/>
@@
 <part name="U$12" library="me433" deviceset="10KOHM-SMD" device=""/>
 <part name="U$18" library="me433" deviceset="10KOHM-SMD" device=""/>
+<part name="U$3" library="me433" deviceset="MCP1702" device=""/>
+<part name="D1" library="me433" deviceset="LED-GREEN" device="0603" value="GREEN"/>
 </parts>
 <sheets>
@@
 <instance part="U$13" gate="G$1" x="22.86" y="7.62"/>
 <instance part="U$14" gate="G$1" x="7.62" y="86.36"/>
-<instance part="D1" gate="G$1" x="27.94" y="38.1" rot="R270"/>
 <instance part="D2" gate="G$1" x="104.14" y="104.14"/>
-<instance part="U$15" gate="G$1" x="58.42" y="96.52"/>
 <instance part="U$17" gate="G$1" x="71.12" y="5.08"/>
 <instance part="J1" gate="G$1" x="-10.16" y="38.1"/>
@@
 <instance part="U$12" gate="G$1" x="25.4" y="66.04"/>
 <instance part="U$18" gate="G$1" x="0" y="7.62"/>
+<instance part="U$3" gate="G$1" x="58.42" y="96.52"/>
+<instance part="D1" gate="G$1" x="25.4" y="38.1" rot="R90"/>
 </instances>
 <busses>
@@
 <net name="VDD" class="0">
 <segment>
-<pinref part="U$15" gate="G$1" pin="VOUT"/>
 <pinref part="U$4" gate="G$1" pin="1"/>
 <wire x1="88.9" y1="101.6" x2="81.28" y2="101.6" width="0.1524" layer="91"/>
@@
 <pinref part="U$10" gate="G$1" pin="+"/>
 <junction x="81.28" y="101.6"/>
+<pinref part="U$3" gate="G$1" pin="VOUT"/>
 </segment>
 <segment>
@@
 <net name="GND" class="0">
 <segment>
-<pinref part="U$15" gate="G$1" pin="VSS"/>
 <wire x1="73.66" y1="91.44" x2="81.28" y2="91.44" width="0.1524" layer="91"/>
 <wire x1="81.28" y1="91.44" x2="81.28" y2="93.98" width="0.1524" layer="91"/>
@@
 <label x="73.66" y="91.44" size="1.778" layer="95"/>
 <pinref part="U$10" gate="G$1" pin="-"/>
+<pinref part="U$3" gate="G$1" pin="VSS"/>
 </segment>
 <segment>
@@
 <wire x1="38.1" y1="38.1" x2="30.48" y2="38.1" width="0.1524" layer="91"/>
 <label x="30.48" y="38.1" size="1.778" layer="95"/>
-<pinref part="D1" gate="G$1" pin="A"/>
+<pinref part="D1" gate="G$1" pin="C"/>
 </segment>
 <segment>
@@
 <net name="N$2" class="0">
 <segment>
-<pinref part="D1" gate="G$1" pin="C"/>
 <pinref part="R1" gate="G$1" pin="2"/>
 <wire x1="20.32" y1="38.1" x2="22.86" y2="38.1" width="0.1524" layer="91"/>
+<pinref part="D1" gate="G$1" pin="A"/>
 </segment>
 </net>
@@
 </segment>
 <segment>
-<pinref part="U$15" gate="G$1" pin="VIN"/>
 <wire x1="43.18" y1="96.52" x2="38.1" y2="96.52" width="0.1524" layer="91"/>
 <label x="38.1" y="96.52" size="1.778" layer="95"/>
 <pinref part="U$5" gate="G$1" pin="1"/>
-</segment>
-<segment>
+<pinref part="U$3" gate="G$1" pin="VIN"/>
+</segment>
+<segment>

Commit message: completed PCB
Parts:
- removed U$3: MCP1702, me433:MCP1702
- added C3: 0.1µF-SMD, me433:0.1µF-SMD
- U$2: value 0.1µF-SMD -> MCP1702; device me433:0.1µF-SMD -> me433:MCP1702
- renumbered D1 to A4, D2 to PWR, U$10 to C6, U$11 to C7, U$12 to R3, U$13 to USER, U$14 to RESET, U$18 to R4, U$4 to C5, U$5 to C4, U$6 to C2, U$7 to C1, U$9 to C8
Connections:
- net 5V: now also U$2.VIN; no longer U$3.VIN
- net GND: now also C3.2, U$2.VSS; no longer U$2.2, U$3.VSS
- net VDD: now also C3.1, U$2.VOUT; no longer U$2.1, U$3.VOUT
