File: HW2/PIC32board/PIC32board.brd (EAGLE design)
At the start: 50 x 50 mm, 24 parts

Commit message: finished adding traces
Parts:
- removed U$15: MCP1702, me433:TO92
- added U$3: MCP1702, me433:TO92
- moved D1 3.81 mm to (2.54, 45.7), turned to 90 degrees
- moved D2 3.81 mm to (6.35, 45.7)
- moved R1 3.81 mm to (2.54, 41.9)
- moved R2 3.81 mm to (6.35, 41.9)
- moved U$4 3.59 mm to (31.8, 41.9), turned to 90 degrees
- moved U$8 2.54 mm to (17.8, 19.1)
- moved U$9 1.27 mm to (35.6, 41.9), turned to 90 degrees
- moved U$18 1.27 mm to (10.2, 12.7), turned to 90 degrees
- turned U$10 to 90 degrees
Connections:
- net 5V: now also U$3.2; no longer U$15.2
- net A4: now also D1.C; no longer D1.A
- net GND: now also U$3.3; no longer U$15.3
- net N$2: now also D1.A; no longer D1.C
- net VDD: now also U$3.1; no longer U$15.1
Routing:
- net GND: track 0.00 -> 136.8 mm
- net VDD: track 0.00 -> 123.8 mm, vias 0 -> 1
- net 5V: track 0.00 -> 94.7 mm, vias 0 -> 1
- net A4: track 0.00 -> 51.7 mm
- net MCLR: track 0.00 -> 45.3 mm, vias 0 -> 1
- net PGED1: track 0.00 -> 33.8 mm
- net PGEC1: track 0.00 -> 33.8 mm
- net B4: track 0.00 -> 33.4 mm, vias 0 -> 2
- net B9: track 0.00 -> 24.8 mm
- net B8: track 0.00 -> 24.8 mm
- net B7: track 0.00 -> 24.8 mm
- net B3: track 0.00 -> 21.4 mm, vias 0 -> 1
- net A1: track 0.00 -> 21.4 mm
- net A0: track 0.00 -> 21.4 mm
- net B2: track 0.00 -> 21.4 mm, vias 0 -> 1
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- added copper zone on layer 1, net GND
- added copper zone on layer 16, net GND

Commit message: completed PCB
Parts:
- removed U$3: MCP1702, me433:TO92
- added C2: 0.1µF-SMD, me433:0603
- U$2: value 0.1µF-SMD -> MCP1702; device me433:0603 -> me433:TO92
- moved U$2 33.9 mm to (22.9, 45.7), turned to 0 degrees
- moved U$17 1.51 mm to (49.5, 42.9)
- renumbered D1 to A4, D2 to PWR, U$10 to C6, U$11 to C7, U$12 to R3, U$13 to USER, U$14 to RESET, U$18 to R4, U$4 to C3, U$5 to C1, U$6 to C5, U$7 to C4, U$9 to C8
Connections:
- net 5V: now also U$2.VIN; no longer U$3.2
- net GND: now also C2.2, U$2.GND; no longer U$2.2, U$3.3
- net VDD: now also C2.1, U$2.VOUT; no longer U$2.1, U$3.1
Routing:
- net GND: track 136.8 -> 112.3 mm
- net VDD: track 123.8 -> 122.0 mm
- net D-: track 28.9 -> 27.4 mm
- net D+: track 30.5 -> 29.3 mm
- net VBUS: track 7.77 -> 8.80 mm
- net ID: track 75.7 -> 75.1 mm
Other:
- board text added: "/Users/allentang1996/Documents/Northwestern/Junior/NUSpring2017/ME 433/northwestern-uni-logo.bmp"
- board text added: "/Users/allentang1996/Downloads/northwestern-uni-logo.bmp"
- board text added: "5V"
- board text added: "A0"
- board text added: "A1"
- board text added: "A4"
- board text added: "Allen Tang ME 433 VER 1.0"
- board text added: "B13"
- board text added: "B14"
- board text added: "B15"
- board text added: "B2"
- board text added: "B3"
- board text added: "B4"
- board text added: "B7"
- board text added: "B8"
- board text added: "B9"
- board text added: "GND"
- board text added: "ON"
- board text added: "VDD"

Commit message: created gerber files
Routing:
- net 5V: track 94.2 -> 93.6 mm
Changed lines of the file:
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@@
 <attribute name="PROD_ID" value="DIO-00821" x="2.54" y="45.72" size="1.778" layer="27" rot="R90" display="off"/>
 </element>
-<element name="U$2" library="me433" package="TO92" value="MCP1702" x="22.86" y="45.72"/>
+<element name="U$2" library="me433" package="TO92" value="MCP1702" x="22.86" y="45.72" smashed="yes"/>
 </elements>
 <signals>
@@
 <wire x1="36.068" y1="6.35" x2="29.21" y2="6.35" width="0.4064" layer="16"/>
 <wire x1="36.068" y1="6.35" x2="48.768" y2="19.05" width="0.4064" layer="16"/>
-<wire x1="18.63" y1="48.26" x2="24.13" y2="48.26" width="0.4064" layer="1"/>
-<wire x1="24.13" y1="48.26" x2="30.48" y2="48.26" width="0.4064" layer="1"/>
+<wire x1="18.63" y1="48.26" x2="23.495" y2="48.26" width="0.4064" layer="1"/>
+<wire x1="23.495" y1="48.26" x2="30.48" y2="48.26" width="0.4064" layer="1"/>
 <wire x1="31.75" y1="46.99" x2="31.75" y2="45.72" width="0.4064" layer="1"/>
 <wire x1="31.75" y1="45.72" x2="34.29" y2="43.18" width="0.4064" layer="1"/>
@@
 <wire x1="29.21" y1="5.5" x2="27.52" y2="3.81" width="0.4064" layer="1"/>
 <contactref element="U$2" pad="VIN"/>
-<wire x1="24.13" y1="48.26" x2="23.495" y2="48.26" width="0.4064" layer="1"/>
 <wire x1="23.495" y1="48.26" x2="22.86" y2="47.625" width="0.4064" layer="1"/>
 </signal>
